File: USB C breadboard power supply.kicad_sch (KiCad schematic)
At the start: 43 parts, among them J1 Conn_02x02_Counter_Clockwise, J2 Conn_02x02_Counter_Clockwise, Q1 IRF9358TRPBF, SW1 SS-10-15SP-LE, U1 CYPD3177-24LQXQT, U2 AP63203WU

Commit message: Update C4 value
Parts:
- C4: value C -> 1uF
Changed lines of the file:
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@@
       (effects (font (size 1.27 1.27)) (justify left))
     )
-    (property "Value" "C" (at 241.3 27.94 0)
+    (property "Value" "1uF" (at 241.3 27.94 0)
       (effects (font (size 1.27 1.27)) (justify left))
     )

Commit message: Updated PCB layout
Reset the layout grid to use 1mm spacing. Changed board outline size. Adjusted copper fill zones and moved them to different layers. Added logo and moved some silkscreen objects.
Other:
- company: (none) -> Byte Sized Engineering
- title: (none) -> USB C Breadboard Power Supply
